File: DataManager.sch (KiCad schematic (older format))
At the start: 37 parts, among them J1 Micro_SD_Card, J2 6P6C, J3 USB_B_Micro, J4 8P8C, J5 8P8C, Q1 MMBT3904, Q2 MMBT3904, U1 ESP32-WROOM-32D, U2 SI8621AB-B-ISR, U3 AP2210-3.3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

Commit message: Board v0.2: Errors fixed
- Pull-up resistor on reset pin
- LS.one (serial) pinout fixed (reversed)
- Isolator U2 RX/TX pinout fixed
- PCB mounting hole diameter enlarged to 3 mm
Parts:
- removed RT1: R_NTC, LibreSolar:R_0603_1608, symbol LibreSolar:R_NTC
- added C11: 2.2u, LibreSolar:C_0603_1608, symbol Project:C
- added R8: 10k, LibreSolar:R_0603_1608, symbol Project:R
- H1, H2, H3, H4: footprint MountingHole:MountingHole_2.5mm -> MountingHole:MountingHole_3mm
- U2: symbol Isolator:ISO7321C -> Project:SI8621AB
Connections:
- net TSENSE is gone; now on net RX_EXT: J2.2
- net +3V3: now also R8.2
- net GND: now also C11.2
- net GND_EXT: now also J2.4; no longer J2.3
- net RESET: now also C11.1, R8.1
- net RX_EXT: now also U2.3 (OUTB); no longer J2.5, U2.2 (OUTA)
- net TX_EXT: now also J2.3, U2.2 (INA); no longer J2.4, U2.3 (INB)
- net U2_RX: now also U2.7 (OUTA); no longer U2.6 (OUTB)
- net U2_TX: now also U2.6 (INB); no longer U2.7 (INA)
- net VCC_EXT: now also J2.1; no longer J2.6
- net BTN: no longer names the net of U1.16 (IO13)
- net BTN: no longer J2.1
- no-connect marks 33 -> 36
Other:
- moved on the sheet: C1
Changed lines of the file:
@@
 EESchema Schematic File Version 4
-LIBS:DataManager-cache
 EELAYER 30 0
 EELAYER END
@@
 Sheet 1 1
 Title "Data Manager"
-Date "2019-09-25"
-Rev "0.1"
+Date "2019-10-17"
+Rev "0.2"
 Comp "Libre Solar"
 Comment1 "Author: Martin Jäger"
@@
 L Project:C C1
 U 1 1 5BD09058
-P 2100 3500
-F 0 "C1" H 2192 3546 50  0000 L CNN
-F 1 "10uF" H 2192 3455 50  0000 L CNN
-F 2 "LibreSolar:C_0805_2012" H 2100 3300 50  0001 C CNN
-F 3 "" H 2125 3575 50  0000 C CNN
-F 4 "Murata" H 2100 3500 50  0001 C CNN "Manufacturer"
-F 5 "GRM21BR61C106KE15L" H 2100 3500 50  0001 C CNN "PartNumber"
-F 6 "16V, X5R" H 2100 3500 50  0001 C CNN "Remarks"
-	1    2100 3500
+P 2100 4200
+F 0 "C1" H 2192 4246 50  0000 L CNN
+F 1 "10uF" H 2192 4155 50  0000 L CNN
+F 2 "LibreSolar:C_0805_2012" H 2100 4000 50  0001 C CNN
+F 3 "" H 2125 4275 50  0000 C CNN
+F 4 "Murata" H 2100 4200 50  0001 C CNN "Manufacturer"
+F 5 "GRM21BR61C106KE15L" H 2100 4200 50  0001 C CNN "PartNumber"
+F 6 "16V, X5R" H 2100 4200 50  0001 C CNN "Remarks"
+	1    2100 4200
 	1    0    0    -1
 $EndComp
@@
 L power:GND #PWR03
 U 1 1 5BD0A3E5
-P 2100 3700
-F 0 "#PWR03" H 2100 3450 50  0001 C CNN
-F 1 "GND" H 2105 3527 50  0000 C CNN
-F 2 "" H 2100 3700 50  0001 C CNN
-F 3 "" H 2100 3700 50  0001 C CNN
-	1    2100 3700
+P 2100 4400
+F 0 "#PWR03" H 2100 4150 50  0001 C CNN
+F 1 "GND" H 2105 4227 50  0000 C CNN
+F 2 "" H 2100 4400 50  0001 C CNN
+F 3 "" H 2100 4400 50  0001 C CNN
+	1    2100 4400
 	1    0    0    -1
 $EndComp
@@
 L power:+3V3 #PWR02
 U 1 1 5BD0A40F
-P 2100 3300
-F 0 "#PWR02" H 2100 3150 50  0001 C CNN
-F 1 "+3V3" H 2115 3473 50  0000 C CNN
-F 2 "" H 2100 3300 50  0001 C CNN
-F 3 "" H 2100 3300 50  0001 C CNN
-	1    2100 3300
-	1    0    0    -1
-$EndComp
-Wire Wire Line
-	2100 3300 2100 3400
-Wire Wire Line
-	2100 3600 2100 3700
+P 2100 4000
+F 0 "#PWR02" H 2100 3850 50  0001 C CNN
+F 1 "+3V3" H 2115 4173 50  0000 C CNN
+F 2 "" H 2100 4000 50  0001 C CNN
+F 3 "" H 2100 4000 50  0001 C CNN
+	1    2100 4000
+	1    0    0    -1
+$EndComp
+Wire Wire Line
+	2100 4000 2100 4100
+Wire Wire Line
+	2100 4300 2100 4400
 $Comp
 L power:+3V3 #PWR0101
@@
 Text Label 4400 3300 2    50   ~ 0
 U2_RX
-Wire Wire Line
-	2800 2300 2400 2300
 NoConn ~ 2800 3600
 NoConn ~ 2800 3700
@@
 L Connector:6P6C J2
 U 1 1 5CE87CF6
-P 2400 7100
-F 0 "J2" H 2457 7667 50  0000 C CNN
-F 1 "6P6C" H 2457 7576 50  0000 C CNN
-F 2 "LibreSolar:RJ12_RJ25_6P6C_Amphenol_54601" V 2400 7125 50  0001 C CNN
-F 3 "~" V 2400 7125 50  0001 C CNN
-F 4 "Amphenol" H 2400 7100 50  0001 C CNN "Manufacturer"
-F 5 "54601-906WPLF" H 2400 7100 50  0001 C CNN "PartNumber"
-	1    2400 7100
-	1    0    0    -1
-$EndComp
-$Comp
-L Isolator:ISO7321C U2
+P 2400 7000
+F 0 "J2" H 2457 7567 50  0000 C CNN
+F 1 "6P6C" H 2457 7476 50  0000 C CNN
+F 2 "LibreSolar:RJ12_RJ25_6P6C_Amphenol_54601" V 2400 7025 50  0001 C CNN
+F 3 "~" V 2400 7025 50  0001 C CNN
+F 4 "Amphenol" H 2400 7000 50  0001 C CNN "Manufacturer"
+F 5 "54601-906WPLF" H 2400 7000 50  0001 C CNN "PartNumber"
+	1    2400 7000
+	1    0    0    1
+$EndComp
+$Comp
+L Project:SI8621AB U2
 U 1 1 5CEB4E0F
 P 5200 7100
@@
 F 1 "SI8621AB-B-ISR" H 5200 7476 50  0000 C CNN
 F 2 "Package_SO:SOIC-8_3.9x4.9mm_P1.27mm" H 5200 6750 50  0001 C CIN
-F 3 "http://www.ti.com/general/docs/lit/getliterature.tsp?genericPartNumber=iso7321c&fileType=pdf" H 5200 7100 50  0001 C CNN
+F 3 "" H 5200 7100 50  0001 C CNN
 	1    5200 7100
 	1    0    0    -1
@@
 	2800 7000 3300 7000
 Wire Wire Line
-	2800 7300 3300 7300
-Wire Wire Line
 	2800 6800 2900 6800
 Wire Wire Line
-	4800 7200 4400 7200
-Wire Wire Line
-	4400 7300 4800 7300
+	4800 7300 4400 7300
+Wire Wire Line
+	4400 7200 4800 7200
 Text Label 3300 6800 2    50   ~ 0
 VCC_EXT
@@
 Text Label 3300 7100 2    50   ~ 0
 GND_EXT
+Text Label 4400 7300 0    50   ~ 0
+RX_EXT
 Text Label 4400 7200 0    50   ~ 0
-RX_EXT
-Text Label 4400 7300 0    50   ~ 0
 TX_EXT
-Text Label 3300 7200 2    50   ~ 0
-TSENSE
-Text Label 3300 7300 2    50   ~ 0
-BTN
 $Comp
 L power:+3V3 #PWR0108
@@
 	6200 7000 5600 7000
 Wire Wire Line
+	5600 7300 6000 7300
+Wire Wire Line
 	5600 7200 6000 7200
-Wire Wire Line
-	5600 7300 6000 7300
+Text Label 6000 7300 2    50   ~ 0
+U2_TX
 Text Label 6000 7200 2    50   ~ 0
-U2_TX
-Text Label 6000 7300 2    50   ~ 0
 U2_RX
 Wire Wire Line
@@
 F 0 "H1" H 9650 10496 50  0000 L CNN
 F 1 "MountingHole" H 9650 10405 50  0000 L CNN
-F 2 "MountingHole:MountingHole_2.5mm" H 9550 10450 50  0001 C CNN
+F 2 "MountingHole:MountingHole_3mm" H 9550 10450 50  0001 C CNN
 F 3 "~" H 9550 10450 50  0001 C CNN
 	1    9550 10450
@@
 F 0 "H2" H 9650 10696 50  0000 L CNN
 F 1 "MountingHole" H 9650 10605 50  0000 L CNN
-F 2 "MountingHole:MountingHole_2.5mm" H 9550 10650 50  0001 C CNN
+F 2 "MountingHole:MountingHole_3mm" H 9550 10650 50  0001 C CNN
 F 3 "~" H 9550 10650 50  0001 C CNN
 	1    9550 10650
@@
 F 0 "H3" H 10750 10496 50  0000 L CNN
 F 1 "MountingHole" H 10750 10405 50  0000 L CNN
-F 2 "MountingHole:MountingHole_2.5mm" H 10650 10450 50  0001 C CNN
+F 2 "MountingHole:MountingHole_3mm" H 10650 10450 50  0001 C CNN
 F 3 "~" H 10650 10450 50  0001 C CNN
 	1    10650 10450
@@
 F 0 "H4" H 10750 10696 50  0000 L CNN
 F 1 "MountingHole" H 10750 10605 50  0000 L CNN
-F 2 "MountingHole:MountingHole_2.5mm" H 10650 10650 50  0001 C CNN
+F 2 "MountingHole:MountingHole_3mm" H 10650 10650 50  0001 C CNN
 F 3 "~" H 10650 10650 50  0001 C CNN
 	1    10650 10650
@@
 	2900 6800 3300 6800
 Wire Wire Line
-	4000 3000 4400 3000
-Text Label 4400 3000 2    50   ~ 0
-BTN
-$Comp
-L LibreSolar:R_NTC RT1
-U 1 1 5DDE11E7
-P 3600 7300
-F 0 "RT1" H 3688 7346 50  0000 L CNN
-F 1 "R_NTC" H 3688 7255 50  0000 L CNN
-F 2 "LibreSolar:R_0603_1608" H 3600 7350 50  0001 C CNN
-F 3 "" H 3600 7350 50  0001 C CNN
-	1    3600 7300
-	1    0    0    -1
-$EndComp
-Wire Wire Line
-	3600 7100 3600 7200
-Wire Wire Line
-	3600 7400 3600 7500
-Wire Wire Line
-	3600 7500 3400 7500
-Wire Wire Line
-	3400 7500 3400 7200
-Wire Wire Line
-	2800 7200 3400 7200
-Wire Wire Line
 	2800 6900 3300 6900
 Wire Wire Line
@@
 Wire Wire Line
 	3600 7100 3600 7000
-Connection ~ 3600 7100
 Wire Wire Line
 	5100 9300 5200 9300
@@
 Text Notes 6400 1600 0    200  ~ 0
 Data Manager - LS.one and LS.bus to WiFi gateway
+$Comp
+L Project:C C11
+U 1 1 5DA8DA09
+P 2100 2500
+F 0 "C11" H 2192 2546 50  0000 L CNN
+F 1 "2.2u" H 2192 2455 50  0000 L CNN
+F 2 "LibreSolar:C_0603_1608" H 2100 2300 50  0001 C CNN
+F 3 "" H 2125 2575 50  0000 C CNN
+	1    2100 2500
+	1    0    0    -1
+$EndComp
+$Comp
+L power:GND #PWR05
+U 1 1 5DA8DF31
+P 2100 2700
+F 0 "#PWR05" H 2100 2450 50  0001 C CNN
+F 1 "GND" H 2105 2527 50  0000 C CNN
+F 2 "" H 2100 2700 50  0001 C CNN
+F 3 "" H 2100 2700 50  0001 C CNN
+	1    2100 2700
+	1    0    0    -1
+$EndComp
+$Comp
+L Project:R R8
+U 1 1 5DAA821F
+P 2100 2100
+F 0 "R8" V 2000 2100 50  0000 C CNN
+F 1 "10k" V 2200 2100 50  0000 C CNN
+F 2 "LibreSolar:R_0603_1608" V 1925 2000 50  0001 C CNN
+F 3 "" H 2100 2100 50  0000 C CNN
+F 4 "Yageo" H 2100 2100 50  0001 C CNN "Manufacturer"
+F 5 "RC0603FR-0710KL" H 2100 2100 50  0001 C CNN "PartNumber"
+	1    2100 2100
+	1    0    0    1
+$EndComp
+$Comp
+L power:+3V3 #PWR01
+U 1 1 5DAB1A59
+P 2100 1900
+F 0 "#PWR01" H 2100 1750 50  0001 C CNN
+F 1 "+3V3" H 2115 2073 50  0000 C CNN
+F 2 "" H 2100 1900 50  0001 C CNN
+F 3 "" H 2100 1900 50  0001 C CNN
+	1    2100 1900
+	1    0    0    -1
+$EndComp
+Wire Wire Line
+	2100 2600 2100 2700
+Wire Wire Line
+	2100 2300 2100 2200
+Wire Wire Line
+	2100 2300 2800 2300
+Wire Wire Line
+	2100 2300 2100 2400
+Connection ~ 2100 2300
+Wire Wire Line
+	2100 2000 2100 1900
+NoConn ~ 2800 7200
+NoConn ~ 2800 7300
+NoConn ~ 4000 3000
 $EndSCHEMATC
